Commit message: add right_finger_joint to URDF for compatibility with ros2_control and MoveIt; mark as passive in SRDF

File: resource/gen3.urdf (robot description, URDF)
Before this commit: robot Gen3, 24 links, 23 joints
Links:
- added link dummy_right_finger_link
Joints:
- added joint right_finger_joint: type fixed, parent robotiq_140_base_link, child dummy_right_finger_link

Commit message: feat: Update gripper model and add new action clients
- Replaced the Robotiq 2F-140 gripper with the Robotiq 2F-85 gripper in the gen3 world file.
- Added a new proto file for the Robotiq 2F-85 gripper, including its geometry and joint configurations.
- Implemented a Python action client for controlling the gripper, allowing for position and effort commands.
- Created a MoveIt action client for planning and executing motion for the manipulator.
- Developed a C++ node to mimic the gripper's finger movements based on joint states.

File: resource/gen3.urdf (robot description, URDF)
Before this commit: robot Gen3, 25 links, 24 joints
Links:
- removed link left_inner_finger
- removed link left_inner_finger_pad
- removed link left_inner_knuckle
- removed link left_outer_finger
- removed link left_outer_knuckle
- removed link right_inner_finger
- removed link right_inner_finger_pad
- removed link right_inner_knuckle
- removed link right_outer_finger
- removed link right_outer_knuckle
- removed link robotiq_140_base_link
- added link robotiq_85_base_link, mass 6.6320197e-01; collision mesh filename=package://robotiq_description/meshes/collision/2f_85/roboti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; visual mesh filename=package://robotiq_description/meshes/visual/2f_85/robotiq_b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
- added link robotiq_85_left_finger_link, mass 4.260376752e-02; collision mesh filename=package://robotiq_description/meshes/collision/2f_85/left_f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; visual mesh filename=package://robotiq_description/meshes/visual/2f_85/left_fing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
- added link robotiq_85_left_finger_tip_link, mass 4.268588744e-02; collision mesh filename=package://robotiq_description/meshes/collision/2f_85/left_f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; visual mesh filename=package://robotiq_description/meshes/visual/2f_85/left_fing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
- added link robotiq_85_left_inner_knuckle_link, mass 2.969376448e-02; collision mesh filename=package://robotiq_description/meshes/collision/2f_85/left_i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; visual mesh filename=package://robotiq_description/meshes/visual/2f_85/left_inne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
- added link robotiq_85_left_knuckle_link, mass 1.384773208e-02; collision mesh filename=package://robotiq_description/meshes/collision/2f_85/left_k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; visual mesh filename=package://robotiq_description/meshes/visual/2f_85/left_knuc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
- added link robotiq_85_right_finger_link, mass 4.260376752000000e-02; collision mesh filename=package://robotiq_description/meshes/collision/2f_85/right_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; visual mesh filename=package://robotiq_description/meshes/visual/2f_85/right_fin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
- added link robotiq_85_right_finger_tip_link, mass 4.268588744e-02; collision mesh filename=package://robotiq_description/meshes/collision/2f_85/right_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; visual mesh filename=package://robotiq_description/meshes/visual/2f_85/right_fin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
- added link robotiq_85_right_inner_knuckle_link, mass 2.969376448e-02; collision mesh filename=package://robotiq_description/meshes/collision/2f_85/right_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; visual mesh filename=package://robotiq_description/meshes/visual/2f_85/right_inn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
- added link robotiq_85_right_knuckle_link, mass 1.384773208e-02; collision mesh filename=package://robotiq_description/meshes/collision/2f_85/right_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; visual mesh filename=package://robotiq_description/meshes/visual/2f_85/right_knu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
Joints:
- removed joint left_inner_finger_joint
- removed joint left_inner_finger_pad_joint
- removed joint left_inner_knuckle_joint
- removed joint left_outer_finger_joint
- removed joint right_inner_finger_joint
- removed joint right_inner_finger_pad_joint
- removed joint right_inner_knuckle_joint
- removed joint right_outer_finger_joint
- removed joint right_outer_knuckle_joint
- removed joint robotiq_140_base_joint
- added joint robotiq_85_base_joint: type fixed, parent robotiq_base_link, child robotiq_85_base_link, origin xyz=0 0 0 rpy=0 0 0
- added joint robotiq_85_left_finger_joint: type fixed, parent robotiq_85_left_knuckle_link, child robotiq_85_left_finger_link, origin xyz=0.03152616 0.0 -0.00376347 rpy=0 0 0
- added joint robotiq_85_left_finger_tip_joint: type continuous, parent robotiq_85_left_finger_link, child robotiq_85_left_finger_tip_link, origin xyz=0.00563134 0.0 0.04718515 rpy=0 0 0, axis 0 -1 0, mimic joint=left_finger_joint multiplier=-1
- added joint robotiq_85_left_inner_knuckle_joint: type continuous, parent robotiq_85_base_link, child robotiq_85_left_inner_knuckle_link, origin xyz=0.0127 0.0 0.06142 rpy=0 0 0, axis 0 -1 0, mimic joint=left_finger_joint
- added joint robotiq_85_right_finger_joint: type fixed, parent robotiq_85_right_knuckle_link, child robotiq_85_right_finger_link, origin xyz=-0.03152616 0.0 -0.00376347 rpy=0 0 0
- added joint robotiq_85_right_finger_tip_joint: type continuous, parent robotiq_85_right_finger_link, child robotiq_85_right_finger_tip_link, origin xyz=-0.00563134 0.0 0.04718515 rpy=0 0 0, axis 0 -1 0, mimic joint=left_finger_joint
- added joint robotiq_85_right_inner_knuckle_joint: type continuous, parent robotiq_85_base_link, child robotiq_85_right_inner_knuckle_link, origin xyz=-0.0127 0.0 0.06142 rpy=0 0 0, axis 0 -1 0, mimic joint=left_finger_joint multiplier=-1
- added joint robotiq_85_right_knuckle_joint: type revolute, parent robotiq_85_base_link, child robotiq_85_right_knuckle_link, origin xyz=-0.03060114 0.0 0.05490452 rpy=0 0 0, axis 0 -1 0, limit lower=-0.8 upper=0.0 effort=50 velocity=0.5, mimic joint=left_finger_joint multiplier=-1
- joint left_finger_joint: axis -1 0 0 -> 0 -1 0; child left_outer_knuckle -> robotiq_85_left_knuckle_link; limit lower=0 upper=0.7 effort=1000 velocity=2.0 -> lower=0.0 upper=0.8 effort=50 velocity=0.5; origin xyz=0 -0.030601 0.054905 rpy=2.2957963267948966 0 0 -> xyz=0.03060114 0.0 0.05490452 rpy=0 0 0; parent robotiq_140_base_link -> robotiq_85_base_link
- joint right_finger_joint: parent robotiq_140_base_link -> robotiq_85_base_link
- joint robotiq_base_joint: origin xyz=0 0 0 rpy=0 0 1.5707963267948966 -> xyz=0 0 0 rpy=0 0 0

Commit message: Enhance robot simulation and control: - Add 'controllers' directory to installation in CMakeLists.txt - Update joint angles in moveit_action_client.py for improved positioning - Introduce gripper_centre joint in URDF and update MoveIt SRDF configuration - Modify kinematics parameters in moveit_kinematics.yaml for better performance - Update gen3.wbt for new object placements and camera configurations - Implement cube_randomizer controller for dynamic cube repositioning - Create BC training configuration in bc_image_joint.yaml - Add complete_episode.py for executing a full episode with IK and cube interaction - Update robomimic dataset metadata for enhanced observation modalities - Implement robomimic_logger for data collection during episodes - Add run_policy.py for policy inference demonstration - Provide training script train_robomimic.sh for BC training setup

File: resource/gen3.urdf (robot description, URDF)
Before this commit: robot Gen3, 25 links, 24 joints
Links:
- added link gripper_centre
Joints:
- added joint gripper_centre_joint: type fixed, parent end_effector_link, child gripper_centre, origin xyz=0 0 0.21 rpy=0 0 0

Commit message: Refine yaw normalization in CubeRandomizer; add single-axis orientation constraint in complete_episode; adjust gripper joint position in URDF; update MoveIt kinematics configuration for local mode and improved rotation scaling

File: resource/gen3.urdf (robot description, URDF)
Before this commit: robot Gen3, 26 links, 25 joints
Joints:
- joint gripper_centre_joint: origin xyz=0 0 0.21 rpy=0 0 0 -> xyz=0 0 0.22 rpy=0 0 0
